Commit message: update package larcc_bringup

File: gripper/urdf/robotiq_arg2f.xacro (robot description, xacro)
@@ -11,5 +11,5 @@
         <origin xyz="0 0 0" rpy="0 0 0" />
         <geometry>
-          <mesh filename="package://robotiq_2f_140_gripper_visualization/meshes/visual/robotiq_arg2f_base_link.stl" />
+          <mesh filename="package://gripper/meshes/visual/robotiq_arg2f_base_link.stl" />
         </geometry>
         <material name="">
@@ -20,5 +20,5 @@
         <origin xyz="0 0 0" rpy="0 0 0" />
         <geometry>
-          <mesh filename="package://robotiq_2f_140_gripper_visualization/meshes/collision/robotiq_arg2f_base_link.stl" />
+          <mesh filename="package://gripper/meshes/collision/robotiq_arg2f_base_link.stl" />
         </geometry>
       </collision>

File: ur_description/urdf/inc/ur_common.xacro (robot description, xacro)
@@ -26,8 +26,8 @@
   <xacro:macro name="read_model_data" params="joint_limits_parameters_file kinematics_parameters_file physical_parameters_file visual_parameters_file">
     <!-- Read .yaml files from disk, load content into properties -->
-    <xacro:property name="joint_limit_parameters" value="${load_yaml(joint_limits_parameters_file)}"/>
-    <xacro:property name="kinematics_parameters" value="${load_yaml(kinematics_parameters_file)}"/>
-    <xacro:property name="physical_parameters" value="${load_yaml(physical_parameters_file)}"/>
-    <xacro:property name="visual_parameters" value="${load_yaml(visual_parameters_file)}"/>
+    <xacro:property name="joint_limit_parameters" value="${xacro.load_yaml(joint_limits_parameters_file)}"/>
+    <xacro:property name="kinematics_parameters" value="${xacro.load_yaml(kinematics_parameters_file)}"/>
+    <xacro:property name="physical_parameters" value="${xacro.load_yaml(physical_parameters_file)}"/>
+    <xacro:property name="visual_parameters" value="${xacro.load_yaml(visual_parameters_file)}"/>
     <!-- Extract subsections from yaml dictionaries -->
     <xacro:property name="limits" value="${joint_limit_parameters['joint_limits']}"/>
