Commit message: gantry xacro update. not yet fully corrected. gantry / tables dimensions and positions require new confirmation in larcc_cell.xacro and gantry.macro.xacro

File: larcc_cell_description/urdf/gantry.macro.xacro (robot description, xacro)
@@ -2,5 +2,5 @@
 <robot name="gantry_macro" xmlns:xacro="http://ros.org/wiki/xacro">
     <!-- A leg macro, to be used bellow by the table macro.-->
-    <xacro:macro name="gantry_leg_macro" params="name parent *origin height leg_radius gantry_thickness">
+    <xacro:macro name="gantry_leg_macro" params="name parent *origin height foot_height leg_radius gantry_thickness">
         <link name="${name}_${parent}">
             <visual>
@@ -41,5 +41,5 @@
     </xacro:macro>
     <!-- A top big beam, to be used bellow by the table macro.-->
-    <xacro:macro name="gantry_big_beam_macro" params="name parent *origin height leg_radius gantry_thickness">
+    <xacro:macro name="gantry_big_beam_macro" params="name parent *origin height foot_height leg_radius gantry_thickness">
         <link name="${name}_gantry">
             <visual>
@@ -80,5 +80,5 @@
     </xacro:macro>
         <!-- A top small beam, to be used bellow by the table macro.-->
-    <xacro:macro name="gantry_small_beam_macro" params="name parent *origin height leg_radius gantry_thickness">
+    <xacro:macro name="gantry_small_beam_macro" params="name parent *origin height foot_height leg_radius gantry_thickness">
         <link name="${name}_${parent}">
             <visual>
@@ -119,5 +119,5 @@
     </xacro:macro>
             <!-- A top small beam, to be used bellow by the table macro.-->
-    <xacro:macro name="gantry_retangular_beam_macro" params="name parent *origin height leg_radius gantry_thickness">
+    <xacro:macro name="gantry_retangular_beam_macro" params="name parent *origin height foot_height leg_radius gantry_thickness">
         <link name="${name}_gantry">
             <visual>
@@ -158,5 +158,5 @@
     </xacro:macro>
     <!-- Table macro, the one that is called from another file.-->
-    <xacro:macro name="gantry_macro" params="name parent *origin width length height
+    <xacro:macro name="gantry_macro" params="name parent *origin width length height foot_height
                                             gantry_thickness leg_radius">
         <!-- %%%%%%%%%%%%%%%%%%%%%%%%%%%%%%%%%%%%%%%%%%%%%-->
@@ -203,70 +203,42 @@
             <parent link="${name}"/>
             <child link="gantry_${name}" />
-            <origin xyz="0 0 ${height}" rpy="0 0 0"/>
+            <origin xyz="0 0 ${height+foot_height}" rpy="0 0 0"/>
         </joint>
         <!-- %%%%%%%%%%%%%%%%%%%%%%%%%%%%%%%%%%%%%%%%%%%%%-->
         <!-- Define the four legs -->
         <!-- %%%%%%%%%%%%%%%%%%%%%%%%%%%%%%%%%%%%%%%%%%%%%-->
-        <xacro:gantry_leg_macro name="leg1" parent="${name}" height="${height}" leg_radius="${leg_radius}" gantry_thickness="${gantry_thickness}">
-            <origin xyz="${-width/2+leg_radius} ${length/2} 0" rpy="0 0 0"/>
-        </xacro:gantry_leg_macro>
-        <xacro:gantry_leg_macro name="leg2" parent="${name}" height="${height}" leg_radius="${leg_radius}" gantry_thickness="${gantry_thickness}">
-            <origin xyz="${width/2} ${length/2} 0" rpy="0 0 0"/>
-        </xacro:gantry_leg_macro>
-        <xacro:gantry_leg_macro name="leg3" parent="${name}" height="${height}" leg_radius="${leg_radius}" gantry_thickness="${gantry_thickness}">
-            <origin xyz="${width/2} ${-length/2-leg_radius} 0" rpy="0 0 0"/>
-        </xacro:gantry_leg_macro>
-        <xacro:gantry_leg_macro name="leg4" parent="${name}" height="${height}" leg_radius="${leg_radius}" gantry_thickness="${gantry_thickness}">
-            <origin xyz="${-width/2+leg_radius} ${-length/2-leg_radius} 0" rpy="0 0 0"/>
-        </xacro:gantry_leg_macro>
-<!--        <xacro:gantry_big_beam_macro name="bigbeam1" parent="${name}" height="${height}" leg_radius="${leg_radius}" gantry_thickness="${gantry_thickness}">-->
-<!--            <origin xyz="${-width/2+leg_radius-1.1/2} ${length/2-0.09} ${height}" rpy="0 0 0"/>-->
-<!--        </xacro:gantry_big_beam_macro>-->
-<!--&lt;!&ndash;&ndash;&gt;-->
-<!--        <xacro:gantry_big_beam_macro name="bigbeam2" parent="${name}" height="${height}" leg_radius="${leg_radius}" gantry_thickness="${gantry_thickness}">-->
-<!--            <origin xyz="${-width/2+leg_radius-1.1/2} ${-length/2+0.09} ${height}" rpy="0 0 0"/>-->
-<!--        </xacro:gantry_big_beam_macro>-->
-        <xacro:gantry_big_beam_macro name="bigbeam1" parent="leg1_gantry" height="${height}" leg_radius="${leg_radius}" gantry_thickness="${gantry_thickness}">
-            <origin xyz="${-(5-width)/2} 0 ${height}" rpy="0 0 0"/>
+        <xacro:gantry_leg_macro name="leg1" parent="${name}" height="${height}" foot_height="${foot_height}" leg_radius="${leg_radius}" gantry_thickness="${gantry_thickness}">
+            <origin xyz="${-width/2-leg_radius} ${length/2} ${foot_height}" rpy="0 0 0"/>
+        </xacro:gantry_leg_macro>
+        <xacro:gantry_leg_macro name="leg2" parent="${name}" height="${height}" foot_height="${foot_height}" leg_radius="${leg_radius}" gantry_thickness="${gantry_thickness}">
+            <origin xyz="${width/2} ${length/2} ${foot_height}" rpy="0 0 0"/>
+        </xacro:gantry_leg_macro>
+        <xacro:gantry_leg_macro name="leg3" parent="${name}" height="${height}" foot_height="${foot_height}" leg_radius="${leg_radius}" gantry_thickness="${gantry_thickness}">
+            <origin xyz="${width/2} ${-length/2-leg_radius} ${foot_height}" rpy="0 0 0"/>
+        </xacro:gantry_leg_macro>
+        <xacro:gantry_leg_macro name="leg4" parent="${name}" height="${height}" foot_height="${foot_height}" leg_radius="${leg_radius}" gantry_thickness="${gantry_thickness}">
+            <origin xyz="${-width/2-leg_radius} ${-length/2-leg_radius} ${foot_height}" rpy="0 0 0"/>
+        </xacro:gantry_leg_macro>
+        <xacro:gantry_big_beam_macro name="bigbeam1" parent="leg1_gantry" height="${height}" foot_height="${foot_height}"  leg_radius="${leg_radius}" gantry_thickness="${gantry_thickness}">
+<!--            <origin xyz="${-(5-width)/2} 0 ${height}" rpy="0 0 0"/>-->
+            <origin xyz="-0.315 0 ${height}" rpy="0 0 0"/>
         </xacro:gantry_big_beam_macro>
-        <xacro:gantry_big_beam_macro name="bigbeam2" parent="leg4_gantry" height="${height}" leg_radius="${leg_radius}" gantry_thickness="${gantry_thickness}">
-            <origin xyz="${-(5-width)/2} 0 ${height}" rpy="0 0 0"/>
+        <xacro:gantry_big_beam_macro name="bigbeam2" parent="leg4_gantry" height="${height}" foot_height="${foot_height}"  leg_radius="${leg_radius}" gantry_thickness="${gantry_thickness}">
+<!--            <origin xyz="${-(5-width)/2} 0 ${height}" rpy="0 0 0"/>-->
+            <origin xyz="-0.315 0 ${height}" rpy="0 0 0"/>
         </xacro:gantry_big_beam_macro>
-<!--        <xacro:gantry_small_beam_macro name="smallbeam1" parent="${name}" height="${height}" leg_radius="${leg_radius}" gantry_thickness="${gantry_thickness}">-->
-<!--            <origin xyz="${-width/2+leg_radius+0.09} ${-length/2-0.5} ${height+0.09}" rpy="0 0 0"/>-->
-<!--        </xacro:gantry_small_beam_macro>-->
-<!--&lt;!&ndash;&ndash;&gt;-->
-<!--        <xacro:gantry_small_beam_macro name="smallbeam2" parent="${name}" height="${height}" leg_radius="${leg_radius}" gantry_thickness="${gantry_thickness}">-->
-<!--            <origin xyz="${width/2-leg_radius+0.09} ${-length/2-0.5} ${height+0.09}" rpy="0 0 0"/>-->
-<!--        </xacro:gantry_small_beam_macro>-->
-<!--        <xacro:gantry_small_beam_macro name="smallbeam1" parent="bigbeam1_gantry" height="${height}" leg_radius="${leg_radius}" gantry_thickness="${gantry_thickness}">-->
-<!--            <origin xyz="${-width/2+leg_radius+0.09} ${-length/2-0.5} ${height+0.09}" rpy="0 0 0"/>-->
-<!--        </xacro:gantry_small_beam_macro>-->
-<!--&lt;!&ndash;&ndash;&gt;-->
-<!--        <xacro:gantry_small_beam_macro name="smallbeam2" parent="bigbeam1_gantry" height="${height}" leg_radius="${leg_radius}" gantry_thickness="${gantry_thickness}">-->
-<!--            <origin xyz="${width/2-leg_radius+0.09} ${-length/2-0.5} ${height+0.09}" rpy="0 0 0"/>-->
-<!--        </xacro:gantry_small_beam_macro>-->
-        <xacro:gantry_small_beam_macro name="smallbeam1" parent="bigbeam1_gantry" height="${height}" leg_radius="${leg_radius}" gantry_thickness="${gantry_thickness}">
+        <xacro:gantry_small_beam_macro name="smallbeam1" parent="bigbeam1_gantry" height="${height}" foot_height="${foot_height}"  leg_radius="${leg_radius}" gantry_thickness="${gantry_thickness}">
             <origin xyz="${(5-width)/2+0.09} ${-((-3.8+length+0.09)/2+3.8)} 0.09" rpy="0 0 0"/>
         </xacro:gantry_small_beam_macro>
-        <xacro:gantry_small_beam_macro name="smallbeam2" parent="bigbeam1_gantry" height="${height}" leg_radius="${leg_radius}" gantry_thickness="${gantry_thickness}">
+        <xacro:gantry_small_beam_macro name="smallbeam2" parent="bigbeam1_gantry" height="${height}" foot_height="${foot_height}"  leg_radius="${leg_radius}" gantry_thickness="${gantry_thickness}">
             <origin xyz="${5-(5-width)/2} ${-((-3.8+length+0.09)/2+3.8)} 0.09" rpy="0 0 0"/>
         </xacro:gantry_small_beam_macro>
-<!--        <xacro:gantry_retangular_beam_macro name="rectangularbeam1" parent="${name}" height="${height}" leg_radius="${leg_radius}" gantry_thickness="${gantry_thickness}">-->
-<!--            <origin xyz="${1+0.045} ${-length/2-0.15} ${height}" rpy="0 ${M_PI/2} 0"/>-->
-<!--        </xacro:gantry_retangular_beam_macro>-->
-<!--        <xacro:gantry_retangular_beam_macro name="rectangularbeam2" parent="${name}" height="${height}" leg_radius="${leg_radius}" gantry_thickness="${gantry_thickness}">-->
-<!--            <origin xyz="${0+0.045} ${-length/2-0.15} ${height}" rpy="0 ${M_PI/2} 0"/>-->
-<!--        </xacro:gantry_retangular_beam_macro>-->
-<!--        <xacro:gantry_retangular_beam_macro name="rectangularbeam3" parent="${name}" height="${height}" leg_radius="${leg_radius}" gantry_thickness="${gantry_thickness}">-->
-<!--            <origin xyz="${-1+0.045} ${-length/2-0.15} ${height}" rpy="0 ${M_PI/2} 0"/>-->
-<!--        </xacro:gantry_retangular_beam_macro>-->
-        <xacro:gantry_retangular_beam_macro name="rectangularbeam1" parent="bigbeam1_gantry" height="${height}" leg_radius="${leg_radius}" gantry_thickness="${gantry_thickness}">
+        <xacro:gantry_retangular_beam_macro name="rectangularbeam1" parent="bigbeam1_gantry" height="${height}" foot_height="${foot_height}"  leg_radius="${leg_radius}" gantry_thickness="${gantry_thickness}">
             <origin xyz="${(5-width)/2+width/4-0.045} -2.8 0" rpy="0 ${M_PI/2} 0"/>
         </xacro:gantry_retangular_beam_macro>
-        <xacro:gantry_retangular_beam_macro name="rectangularbeam2" parent="bigbeam1_gantry" height="${height}" leg_radius="${leg_radius}" gantry_thickness="${gantry_thickness}">
+        <xacro:gantry_retangular_beam_macro name="rectangularbeam2" parent="bigbeam1_gantry" height="${height}" foot_height="${foot_height}"  leg_radius="${leg_radius}" gantry_thickness="${gantry_thickness}">
             <origin xyz="${(5-width)/2+width/2-0.045} -2.8 0" rpy="0 ${M_PI/2} 0"/>
         </xacro:gantry_retangular_beam_macro>
-        <xacro:gantry_retangular_beam_macro name="rectangularbeam3" parent="bigbeam1_gantry" height="${height}" leg_radius="${leg_radius}" gantry_thickness="${gantry_thickness}">
+        <xacro:gantry_retangular_beam_macro name="rectangularbeam3" parent="bigbeam1_gantry" height="${height}" foot_height="${foot_height}"  leg_radius="${leg_radius}" gantry_thickness="${gantry_thickness}">
             <origin xyz="${(5-width)/2+3*width/4-0.045} -2.8 0" rpy="0 ${M_PI/2} 0"/>
         </xacro:gantry_retangular_beam_macro>

File: larcc_cell_description/urdf/larcc_cell.xacro (robot description, xacro)
@@ -10,4 +10,6 @@
     <!-- Gantry properties-->
     <xacro:property name="gantry_height" value="2.29"/>
+    <xacro:property name="gantry_foot_height" value="0.065"/>
+<!--    <xacro:property name="gantry_height" value="2.353"/>-->
     <xacro:property name="gantry_width" value="4"/>
     <xacro:property name="gantry_length" value="2.8"/>
@@ -25,5 +27,5 @@
 <!--    Place gantry-->
     <xacro:gantry_macro name="gantry" parent="world" width="${gantry_width}"
-                        length="${gantry_length}" height="${gantry_height}"
+                        length="${gantry_length}" height="${gantry_height}" foot_height="${gantry_foot_height}"
                         gantry_thickness="${gantry_thickness}" leg_radius="${gantry_leg_radius}">
         <origin xyz="0 0 0" rpy="0 0 0"/>

Commit message: larccell xacro: gantry is now corrected wrt /world. tables+robot still need to be corrected. robot wrt cameras is fixed and calibrated.

File: larcc_cell_description/urdf/gantry.macro.xacro (robot description, xacro)
@@ -209,5 +209,5 @@
         <!-- %%%%%%%%%%%%%%%%%%%%%%%%%%%%%%%%%%%%%%%%%%%%%-->
         <xacro:gantry_leg_macro name="leg1" parent="${name}" height="${height}" foot_height="${foot_height}" leg_radius="${leg_radius}" gantry_thickness="${gantry_thickness}">
-            <origin xyz="${-width/2-leg_radius} ${length/2} ${foot_height}" rpy="0 0 0"/>
+            <origin xyz="${-(width/2)-leg_radius} ${length/2} ${foot_height}" rpy="0 0 0"/>
         </xacro:gantry_leg_macro>
         <xacro:gantry_leg_macro name="leg2" parent="${name}" height="${height}" foot_height="${foot_height}" leg_radius="${leg_radius}" gantry_thickness="${gantry_thickness}">
@@ -215,8 +215,8 @@
         </xacro:gantry_leg_macro>
         <xacro:gantry_leg_macro name="leg3" parent="${name}" height="${height}" foot_height="${foot_height}" leg_radius="${leg_radius}" gantry_thickness="${gantry_thickness}">
-            <origin xyz="${width/2} ${-length/2-leg_radius} ${foot_height}" rpy="0 0 0"/>
+            <origin xyz="${width/2} ${-(length/2)-leg_radius} ${foot_height}" rpy="0 0 0"/>
         </xacro:gantry_leg_macro>
         <xacro:gantry_leg_macro name="leg4" parent="${name}" height="${height}" foot_height="${foot_height}" leg_radius="${leg_radius}" gantry_thickness="${gantry_thickness}">
-            <origin xyz="${-width/2-leg_radius} ${-length/2-leg_radius} ${foot_height}" rpy="0 0 0"/>
+            <origin xyz="${-(width/2)-leg_radius} ${-(length/2)-leg_radius} ${foot_height}" rpy="0 0 0"/>
         </xacro:gantry_leg_macro>
         <xacro:gantry_big_beam_macro name="bigbeam1" parent="leg1_gantry" height="${height}" foot_height="${foot_height}"  leg_radius="${leg_radius}" gantry_thickness="${gantry_thickness}">
@@ -229,17 +229,17 @@
         </xacro:gantry_big_beam_macro>
         <xacro:gantry_small_beam_macro name="smallbeam1" parent="bigbeam1_gantry" height="${height}" foot_height="${foot_height}"  leg_radius="${leg_radius}" gantry_thickness="${gantry_thickness}">
-            <origin xyz="${(5-width)/2+0.09} ${-((-3.8+length+0.09)/2+3.8)} 0.09" rpy="0 0 0"/>
+            <origin xyz="${0.32+leg_radius} ${-(length+leg_radius+0.37)} ${leg_radius}" rpy="0 0 0"/>
         </xacro:gantry_small_beam_macro>
         <xacro:gantry_small_beam_macro name="smallbeam2" parent="bigbeam1_gantry" height="${height}" foot_height="${foot_height}"  leg_radius="${leg_radius}" gantry_thickness="${gantry_thickness}">
-            <origin xyz="${5-(5-width)/2} ${-((-3.8+length+0.09)/2+3.8)} 0.09" rpy="0 0 0"/>
+            <origin xyz="${0.32+leg_radius+leg_radius+width} ${-(length+leg_radius+0.37)} ${leg_radius}" rpy="0 0 0"/>
         </xacro:gantry_small_beam_macro>
         <xacro:gantry_retangular_beam_macro name="rectangularbeam1" parent="bigbeam1_gantry" height="${height}" foot_height="${foot_height}"  leg_radius="${leg_radius}" gantry_thickness="${gantry_thickness}">
-            <origin xyz="${(5-width)/2+width/4-0.045} -2.8 0" rpy="0 ${M_PI/2} 0"/>
+            <origin xyz="${0.32+leg_radius+0.98+0.045} ${-(length+leg_radius+0.12)} 0" rpy="0 ${M_PI/2} 0"/>
         </xacro:gantry_retangular_beam_macro>
         <xacro:gantry_retangular_beam_macro name="rectangularbeam2" parent="bigbeam1_gantry" height="${height}" foot_height="${foot_height}"  leg_radius="${leg_radius}" gantry_thickness="${gantry_thickness}">
-            <origin xyz="${(5-width)/2+width/2-0.045} -2.8 0" rpy="0 ${M_PI/2} 0"/>
+            <origin xyz="${0.32+leg_radius+0.98+0.045+0.945+0.045} ${-(length+leg_radius+0.12)} 0" rpy="0 ${M_PI/2} 0"/>
         </xacro:gantry_retangular_beam_macro>
         <xacro:gantry_retangular_beam_macro name="rectangularbeam3" parent="bigbeam1_gantry" height="${height}" foot_height="${foot_height}"  leg_radius="${leg_radius}" gantry_thickness="${gantry_thickness}">
-            <origin xyz="${(5-width)/2+3*width/4-0.045} -2.8 0" rpy="0 ${M_PI/2} 0"/>
+            <origin xyz="${0.32+leg_radius+0.98+0.045+0.945+0.045+0.955+0.045} ${-(length+leg_radius+0.12)} 0" rpy="0 ${M_PI/2} 0"/>
         </xacro:gantry_retangular_beam_macro>
     </xacro:macro>

File: larcc_cell_description/urdf/larcc_cell.xacro (robot description, xacro)
@@ -13,5 +13,5 @@
 <!--    <xacro:property name="gantry_height" value="2.353"/>-->
     <xacro:property name="gantry_width" value="4"/>
-    <xacro:property name="gantry_length" value="2.8"/>
+    <xacro:property name="gantry_length" value="2.7975"/>
     <xacro:property name="gantry_thickness" value="0"/>
     <xacro:property name="gantry_leg_radius" value="0.09"/>
