Commit message: added and calibrated orbbec astra pro

File: larcc_cell_description/urdf/astra.urdf.xacro (robot description, xacro)
@@ -17,5 +17,5 @@
         <origin xyz="-0.03 -0.06 0" rpy="${pi} 0 ${pi/2}"/>
         <geometry>
-          <mesh filename="package://larcc_description/meshes/sensors/astra2.dae" scale="${scale}"/>
+          <mesh filename="package://larcc_cell_description/meshes/sensors/astra2.dae" scale="${scale}"/>
         </geometry>
       </visual>

File: larcc_cell_description/urdf/larcc_cell.xacro (robot description, xacro)
@@ -19,4 +19,5 @@
     <xacro:include filename="$(find ur_description)/urdf/inc/ur10e_macro.xacro"/>
     <xacro:include filename="$(find realsense2_description)/urdf/test_d435i_camera.urdf.xacro" />
+    <xacro:include filename="$(find larcc_cell_description)/urdf/astra.urdf.xacro"/>
     <xacro:include filename="$(find gripper)/urdf/robotiq_arg2f_140_model_macro.xacro" />
     <xacro:include filename="$(find larcc_cell_description)/urdf/table.macro.xacro"/>
@@ -39,4 +40,9 @@
         <origin xyz="-0.161 0.222 1.210" rpy="3.210079633 2.720592654 2.809"/>
     </xacro:realsense2_camera>
+    <!-- Astra below was not well calibrated -->
+    <xacro:sensor_astra prefix="camera_4" parent="world" scale="1 1 1">
+        <origin xyz="0.8891137 1.18206377 2.31900029"
+                rpy="-0.10196342984026999 0.5145692159638564 -1.7990340284545345"/>
+    </xacro:sensor_astra>
     <joint name="tool0-FT_sensor_base" type="fixed">
         <parent link="tool0"/>

Commit message: Adjustments to xacro files (new camera pose and names for atom rgb extrinsic calibration)

File: larcc_cell_description/urdf/astra.urdf.xacro (robot description, xacro)
@@ -38,16 +38,4 @@
       <selfCollide>false</selfCollide>
     </gazebo>
-    <joint name="${prefix}_rgb_joint" type="fixed">
-      <origin xyz="0 -0.045 0" rpy="0 0 0" />
-      <parent link="${prefix}_link"/>
-      <child link="${prefix}_rgb_frame" />
-    </joint>
-    <link name="${prefix}_rgb_frame"/>
-    <joint name="${prefix}_rgb_optical_joint" type="fixed">
-      <origin xyz="0 0 0" rpy="${-pi/2} 0 ${-pi/2}" />
-      <parent link="${prefix}_rgb_frame" />
-      <child link="${prefix}_rgb_optical_frame" />
-    </joint>
-    <link name="${prefix}_rgb_optical_frame"/>
     <joint name="${prefix}_depth_joint" type="fixed">
         <origin xyz="0 -0.02 0" rpy="0 0 0" />
@@ -83,11 +71,11 @@
                   <alwaysOn>true</alwaysOn>
                   <updateRate>0</updateRate>
-                  <imageTopicName>rgb/image_raw</imageTopicName>
+                  <imageTopicName>color/image_raw</imageTopicName>
                   <depthImageTopicName>depth/image_raw</depthImageTopicName>
                   <pointCloudTopicName>depth/points</pointCloudTopicName>
-                  <cameraInfoTopicName>rgb/camera_info</cameraInfoTopicName>
+                  <cameraInfoTopicName>color/camera_info</cameraInfoTopicName>
                   <depthImageCameraInfoTopicName>depth/camera_info</depthImageCameraInfoTopicName>
 <!--                  <frameName>${prefix}_depth_optical_frame</frameName>-->
-                  <frameName>${prefix}_rgb_optical_frame</frameName>
+                  <frameName>${prefix}_color_optical_frame</frameName>
 <!--                  <frameName>${prefix}_link</frameName>-->
                   <baseline>0.1</baseline>

File: larcc_cell_description/urdf/larcc_cell.xacro (robot description, xacro)
@@ -37,6 +37,8 @@
     </joint>
 <!--    Place d45i camera-->
+<!--    Note: should add Pi value (3.14159) to second rotation value (p)-->
     <xacro:realsense2_camera parent="world" use_nominal_extrinsics="true">
-        <origin xyz="-0.161 0.222 1.210" rpy="3.210079633 2.720592654 2.809"/>
+<!--        <origin xyz="-0.161 0.222 1.210" rpy="3.210079633 2.720592654 2.809"/>-->
+        <origin xyz="-0.507 0.222 1.312" rpy="3.107 2.5559 -3.080"/>
     </xacro:realsense2_camera>
 <!--    &lt;!&ndash; Astra below was not well calibrated &ndash;&gt;-->

File: realsense2_description/urdf/test_d435i_camera.urdf.xacro (robot description, xacro)
@@ -5,5 +5,5 @@
   <xacro:macro name="realsense2_camera" params="parent *origin name:=camera use_nominal_extrinsics">
 <!--    <xacro:sensor_d435i parent="${parent}" origin="origin" use_nominal_extrinsics="$(arg use_nominal_extrinsics)">-->
-    <xacro:sensor_d435i parent="${parent}" origin="origin" use_nominal_extrinsics="${use_nominal_extrinsics}">
+    <xacro:sensor_d435i parent="${parent}" name="${name}" origin="origin" use_nominal_extrinsics="${use_nominal_extrinsics}">
 <!--      <origin xyz="0 0 0" rpy="0 0 0"/>-->
     </xacro:sensor_d435i>

Commit message: fix astra urdf!!! larcc_cell.xacro updated

File: larcc_cell_description/urdf/astra.urdf.xacro (robot description, xacro)
@@ -2,29 +2,27 @@
 <robot name="sensor_astra" xmlns:xacro="http://ros.org/wiki/xacro">
   <!-- Xacro properties -->
-  <xacro:property name="astra_cam_py" value="-0.0125"/>
-  <xacro:property name="astra_depth_rel_rgb_py" value="0.0250" />
-  <xacro:property name="astra_cam_rel_rgb_py"   value="-0.0125" />
-  <xacro:property name="astra_dae_display_scale"   value="0.1" />
+  <xacro:property name="astra_depth_rel_cam_py" value="0.0370" />
+  <xacro:property name="astra_cam_rel_rgb_py"   value="0.0100" />
+  <xacro:property name="astra_dae_display_scale"   value="1" />
   <!-- Parameterised in part by the values in turtlebot_properties.urdf.xacro -->
-  <xacro:macro name="sensor_astra" params="parent prefix *origin scale">
-    <joint name="${prefix}_joint" type="fixed">
+  <xacro:macro name="sensor_astra" params="parent prefix *origin">
+    <joint name="${prefix}_rgb_joint" type="fixed">
       <xacro:insert_block name="origin" />
       <parent link="${parent}"/>
-      <child link="${prefix}_link"/>
+      <child link="${prefix}_link" />
     </joint>
     <link name="${prefix}_link">
       <visual>
-        <origin xyz="-0.03 -0.06 0" rpy="${pi} 0 ${pi/2}"/>
+        <origin xyz="0 0 0" rpy="${M_PI/2} 0 ${M_PI/2}"/>
         <geometry>
-          <mesh filename="package://larcc_cell_description/meshes/sensors/astra2.dae" scale="${scale}"/>
+          <mesh filename="package://larcc_cell_description/meshes/sensors/astra2.dae" scale="${astra_dae_display_scale} ${astra_dae_display_scale} ${astra_dae_display_scale}"/>
         </geometry>
       </visual>
-<!--      <collision>-->
-<!--        &lt;!&ndash; <origin xyz="0.0 0.0 0.0" rpy="0 0 0" /> &ndash;&gt;-->
-<!--        <origin xyz="-0.01 -0.06 0" rpy="0 0 0"/>-->
-<!--        <geometry>-->
-<!--        <box size="0.0400 0.1650 0.0300"/>-->
-<!--      </geometry>-->
-<!--      </collision>-->
+      <collision>
+        <origin xyz="0.0 0.0 0.0" rpy="0 0 0" />
+        <geometry>
+        <box size="0.0400 0.1650 0.0300"/>
+      </geometry>
+      </collision>
       <inertial>
         <mass value="0.564" />
@@ -35,58 +33,17 @@
       </inertial>
     </link>
-    <gazebo reference="${prefix}_link">
-      <selfCollide>false</selfCollide>
-    </gazebo>
+    <joint name="${prefix}_joint" type="fixed">
+      <origin xyz="0 ${astra_cam_rel_rgb_py} 0"
+              rpy="0 0 0"/>
+      <parent link="${prefix}_link"/>
+      <child link="${prefix}_rgb_optical_frame"/>
+    </joint>
+    <link name="${prefix}_rgb_optical_frame"/>
     <joint name="${prefix}_depth_joint" type="fixed">
-        <origin xyz="0 -0.02 0" rpy="0 0 0" />
-        <parent link="${prefix}_link" />
-        <child link="${prefix}_depth_frame" />
-    </joint>
-    <link name="${prefix}_depth_frame"/>
-    <joint name="${prefix}_depth_optical_joint" type="fixed">
-        <origin xyz="0 0 0" rpy="${-pi/2} 0 ${-pi/2}" />
-        <parent link="${prefix}_depth_frame" />
-        <child link="${prefix}_depth_optical_frame" />
+      <origin xyz="0 ${astra_depth_rel_cam_py} 0" rpy="0 0 0" />
+      <parent link="${prefix}_link" />
+      <child link="${prefix}_depth_optical_frame" />
     </joint>
     <link name="${prefix}_depth_optical_frame"/>
-     <gazebo reference="${prefix}_depth_frame">
-          <sensor type="depth" name="camera">
-              <always_on>true</always_on>
-              <update_rate>8.0</update_rate>
-              <camera>
-                  <horizontal_fov>${60.0*pi/180.0}</horizontal_fov>
-                  <image>
-                      <format>B8G8R8</format>
-<!--                      <format>RGB_INT8</format>-->
-                      <width>1280</width>
-                      <height>800</height>
-                  </image>
-                  <clip>
-                      <near>0.10</near>
-                      <far>8.0</far>
-                  </clip>
-              </camera>
-              <plugin name="${prefix}_camera_controller" filename="libgazebo_ros_openni_kinect.so">
-                  <cameraName>${prefix}</cameraName>
-                  <alwaysOn>true</alwaysOn>
-                  <updateRate>0</updateRate>
-                  <imageTopicName>color/image_raw</imageTopicName>
-                  <depthImageTopicName>depth/image_raw</depthImageTopicName>
-                  <pointCloudTopicName>depth/points</pointCloudTopicName>
-                  <cameraInfoTopicName>color/camera_info</cameraInfoTopicName>
-                  <depthImageCameraInfoTopicName>depth/camera_info</depthImageCameraInfoTopicName>
-<!--                  <frameName>${prefix}_depth_optical_frame</frameName>-->
-                  <frameName>${prefix}_color_optical_frame</frameName>
-<!--                  <frameName>${prefix}_link</frameName>-->
-                  <baseline>0.1</baseline>
-                  <distortion_k1>0.0</distortion_k1>
-                  <distortion_k2>0.0</distortion_k2>
-                  <distortion_k3>0.0</distortion_k3>
-                  <distortion_t1>0.0</distortion_t1>
-                  <distortion_t2>0.0</distortion_t2>
-                  <pointCloudCutoff>0.4</pointCloudCutoff>
-              </plugin>
-          </sensor>
-      </gazebo>
   </xacro:macro>
 </robot>

File: larcc_cell_description/urdf/larcc_cell.xacro (robot description, xacro)
@@ -42,9 +42,9 @@
         <origin xyz="-0.507 0.222 1.312" rpy="3.107 2.5559 -3.080"/>
     </xacro:realsense2_camera>
-<!--    &lt;!&ndash; Astra below was not well calibrated &ndash;&gt;-->
-<!--    <xacro:sensor_astra prefix="camera_4" parent="world" scale="1 1 1">-->
-<!--        <origin xyz="0.8891137 1.18206377 2.31900029"-->
-<!--                rpy="-0.10196342984026999 0.5145692159638564 -1.7990340284545345"/>-->
-<!--    </xacro:sensor_astra>-->
+    <!-- Astra below was not well calibrated -->
+    <xacro:sensor_astra prefix="camera_4" parent="world">
+        <origin xyz="0.8891137 1.18206377 2.31900029"
+                rpy="-0.10196342984026999 0.5145692159638564 -1.7990340284545345"/>
+    </xacro:sensor_astra>
     <joint name="tool0-FT_sensor_base" type="fixed">
         <parent link="tool0"/>

Commit message: restore gazebo section to astra.urdf.xacro

File: larcc_cell_description/urdf/astra.urdf.xacro (robot description, xacro)
@@ -34,6 +34,5 @@
     </link>
     <joint name="${prefix}_joint" type="fixed">
-      <origin xyz="0 ${astra_cam_rel_rgb_py} 0"
-              rpy="0 0 0"/>
+      <origin xyz="0 ${astra_cam_rel_rgb_py} 0" rpy="0 0 0"/>
       <parent link="${prefix}_link"/>
       <child link="${prefix}_rgb_optical_frame"/>
@@ -46,4 +45,43 @@
     </joint>
     <link name="${prefix}_depth_optical_frame"/>
+    <gazebo reference="${prefix}_depth_frame">
+          <sensor type="depth" name="camera">
+              <always_on>true</always_on>
+              <update_rate>8.0</update_rate>
+              <camera>
+                  <horizontal_fov>${60.0*pi/180.0}</horizontal_fov>
+                  <image>
+                      <format>B8G8R8</format>
+<!--                      <format>RGB_INT8</format>-->
+                      <width>640</width>
+                      <height>480</height>
+                  </image>
+                  <clip>
+                      <near>0.10</near>
+                      <far>8.0</far>
+                  </clip>
+              </camera>
+              <plugin name="${prefix}_camera_controller" filename="libgazebo_ros_openni_kinect.so">
+                  <cameraName>${prefix}</cameraName>
+                  <alwaysOn>true</alwaysOn>
+                  <updateRate>0</updateRate>
+                  <imageTopicName>color/image_raw</imageTopicName>
+                  <depthImageTopicName>depth/image_raw</depthImageTopicName>
+                  <pointCloudTopicName>depth/points</pointCloudTopicName>
+                  <cameraInfoTopicName>color/camera_info</cameraInfoTopicName>
+                  <depthImageCameraInfoTopicName>depth/camera_info</depthImageCameraInfoTopicName>
+<!--                  <frameName>${prefix}_depth_optical_frame</frameName>-->
+                  <frameName>${prefix}_color_optical_frame</frameName>
+<!--                  <frameName>${prefix}_link</frameName>-->
+                  <baseline>0.1</baseline>
+                  <distortion_k1>0.0</distortion_k1>
+                  <distortion_k2>0.0</distortion_k2>
+                  <distortion_k3>0.0</distortion_k3>
+                  <distortion_t1>0.0</distortion_t1>
+                  <distortion_t2>0.0</distortion_t2>
+                  <pointCloudCutoff>0.4</pointCloudCutoff>
+              </plugin>
+          </sensor>
+      </gazebo>
   </xacro:macro>
 </robot>

Commit message: astra TF's fixed (camera_link & optical_frames) Gripper open and close alias fixed

File: larcc_cell_description/urdf/astra.urdf.xacro (robot description, xacro)
@@ -14,5 +14,5 @@
     <link name="${prefix}_link">
       <visual>
-        <origin xyz="0 0 0" rpy="${M_PI/2} 0 ${M_PI/2}"/>
+        <origin xyz="0 0 0" rpy="0 ${M_PI} ${-M_PI/2}"/>
         <geometry>
           <mesh filename="package://larcc_cell_description/meshes/sensors/astra2.dae" scale="${astra_dae_display_scale} ${astra_dae_display_scale} ${astra_dae_display_scale}"/>
@@ -34,5 +34,5 @@
     </link>
     <joint name="${prefix}_joint" type="fixed">
-      <origin xyz="0 ${astra_cam_rel_rgb_py} 0" rpy="0 0 0"/>
+      <origin xyz="0 ${astra_cam_rel_rgb_py} 0" rpy="${M_PI/2} ${M_PI} ${M_PI/2}"/>
       <parent link="${prefix}_link"/>
       <child link="${prefix}_rgb_optical_frame"/>
@@ -40,5 +40,5 @@
     <link name="${prefix}_rgb_optical_frame"/>
     <joint name="${prefix}_depth_joint" type="fixed">
-      <origin xyz="0 ${astra_depth_rel_cam_py} 0" rpy="0 0 0" />
+      <origin xyz="0 ${astra_depth_rel_cam_py} 0" rpy="${M_PI/2} ${M_PI} ${M_PI/2}" />
       <parent link="${prefix}_link" />
       <child link="${prefix}_depth_optical_frame" />

File: larcc_cell_description/urdf/larcc_cell.xacro (robot description, xacro)
@@ -50,5 +50,5 @@
     <xacro:sensor_astra prefix="camera_top" parent="world">
         <origin xyz="0.1 0 2.41900029"
-                rpy="0 ${M_PI} 0"/>
+                rpy="0 0 0"/>
     </xacro:sensor_astra>
 <!--    &lt;!&ndash; Astra top before calibration &ndash;&gt;-->

Commit message: corrected table_beam (bosch 40x40 and not minitec 45x45). Also, added new collisions to this table_beam. Astra cameras collisions also corrected. All of this on larcc_cell.xacro.

File: larcc_cell_description/urdf/astra.urdf.xacro (robot description, xacro)
@@ -20,5 +20,5 @@
       </visual>
       <collision>
-        <origin xyz="0.0 0.0 0.0" rpy="0 0 0" />
+        <origin xyz="0.02 0.0 0.0" rpy="0 0 0" />
         <geometry>
         <box size="0.0400 0.1650 0.0300"/>

File: larcc_cell_description/urdf/larcc_cell.xacro (robot description, xacro)
@@ -123,12 +123,12 @@
             <origin xyz="0.0 0.0 0.0" rpy="0 0 0" />
             <geometry>
-                <mesh filename="package://larcc_cell_description/meshes/minitec_45x45_1500.STL" scale="0.001 0.001 0.001" />
+                <mesh filename="package://larcc_cell_description/meshes/bosch_40x40x150.STL" scale="0.001 0.01 0.001" />
             </geometry>
             <material name="grey"/>
         </visual>
         <collision>
-            <origin xyz="0 0 0" rpy="0 0 0" />
+            <origin xyz="0.02 0.75 0.02" rpy="${M_PI/2} 0 0" />
             <geometry>
-                <box size="0.045 0.045 1.5"/>
+                <box size="0.05 0.05 1.55"/>
             </geometry>
         </collision>
@@ -144,5 +144,5 @@
         <parent link="table_base" />
         <child link="table_beam" />
-        <origin xyz="0.305 -0.625 0.0025" rpy="${M_PI/2} 0 0"/>
+        <origin xyz="0.308 -0.625 0.0035" rpy="${M_PI/2} 0 0"/>
     </joint>
      <!-- Collision box representing the ceiling -->
