Commit message: Gripper Action Server fully working UR10eArm class working to control manipulator (from /world to /end_effector) ActionClient working to control manipulator, but only for joint states. Actions still dont work to tcp pose goals.

File: larcc_cell_description/urdf/larcc_cell.xacro (robot description, xacro)
@@ -36,5 +36,5 @@
     </joint>
 <!--    Place d45i camera-->
-<!--    <xacro:realsense2_camera parent="base_link" use_nominal_extrinsics="true">-->
+<!--    <xacro:realsense2_camera parent="base" use_nominal_extrinsics="true">-->
 <!--        <origin xyz="0.797 -0.803 0.432" rpy="3.135 2.462 -1.577"/>-->
 <!--    </xacro:realsense2_camera>-->
@@ -86,4 +86,10 @@
         <origin xyz="0 0 0.011" rpy="0 0 0"/>
     </joint>
+    <link name="end_effector"/>
+    <joint name="gripper-end_effector" type="fixed">
+        <parent link="robotiq_arg2f_base_link"/>
+        <child link="end_effector"/>
+        <origin xyz="0.0007295637845960989 0.0009607961805311316 0.21573113136562894" rpy="0 -0.001546440756787199 -1.572652377645297"/>
+    </joint>
 <!--    Place base table-->
     <xacro:table_macro name="table_base" parent="world" width="${table_width}"

Commit message: Adding realsense2_description package to import urdf model of IntelRealsense Manual Calibration already performed

File: larcc_cell_description/urdf/larcc_cell.xacro (robot description, xacro)
@@ -18,5 +18,5 @@
     <xacro:include filename="$(find larcc_cell_description)/urdf/properties.xacro"/>
     <xacro:include filename="$(find ur_description)/urdf/inc/ur10e_macro.xacro"/>
-<!--    <xacro:include filename="$(find realsense2_description)/urdf/test_d435i_camera.urdf.xacro" />-->
+    <xacro:include filename="$(find realsense2_description)/urdf/test_d435i_camera.urdf.xacro" />
     <xacro:include filename="$(find gripper)/urdf/robotiq_arg2f_140_model_macro.xacro" />
     <xacro:include filename="$(find larcc_cell_description)/urdf/table.macro.xacro"/>
@@ -36,7 +36,8 @@
     </joint>
 <!--    Place d45i camera-->
-<!--    <xacro:realsense2_camera parent="base" use_nominal_extrinsics="true">-->
-<!--        <origin xyz="0.797 -0.803 0.432" rpy="3.135 2.462 -1.577"/>-->
-<!--    </xacro:realsense2_camera>-->
+    <xacro:realsense2_camera parent="world" use_nominal_extrinsics="true">
+<!--        <origin xyz="0.808 0.160 1.201" rpy="-3.092 0.390 -2.716"/>-->
+        <origin xyz="0.808 0.160 1.201" rpy="0.049592654 0.390 -2.716"/>
+    </xacro:realsense2_camera>
     <joint name="tool0-FT_sensor_base" type="fixed">
         <parent link="tool0"/>

Commit message: realsense2_camera manual calibration DONE Remember: you have to add pi to 2nd value of rotation (p in rpy).

File: larcc_cell_description/urdf/larcc_cell.xacro (robot description, xacro)
@@ -37,6 +37,5 @@
 <!--    Place d45i camera-->
     <xacro:realsense2_camera parent="world" use_nominal_extrinsics="true">
-<!--        <origin xyz="0.808 0.160 1.201" rpy="-3.092 0.390 -2.716"/>-->
-        <origin xyz="0.808 0.160 1.201" rpy="0.049592654 0.390 -2.716"/>
+        <origin xyz="-0.161 0.222 1.210" rpy="3.210079633 2.720592654 2.809"/>
     </xacro:realsense2_camera>
     <joint name="tool0-FT_sensor_base" type="fixed">

Commit message: commit

File: larcc_cell_description/urdf/larcc_cell.xacro (robot description, xacro)
@@ -40,9 +40,9 @@
         <origin xyz="-0.161 0.222 1.210" rpy="3.210079633 2.720592654 2.809"/>
     </xacro:realsense2_camera>
-    <!-- Astra below was not well calibrated -->
-    <xacro:sensor_astra prefix="camera_4" parent="world" scale="1 1 1">
-        <origin xyz="0.8891137 1.18206377 2.31900029"
-                rpy="-0.10196342984026999 0.5145692159638564 -1.7990340284545345"/>
-    </xacro:sensor_astra>
+<!--    &lt;!&ndash; Astra below was not well calibrated &ndash;&gt;-->
+<!--    <xacro:sensor_astra prefix="camera_4" parent="world" scale="1 1 1">-->
+<!--        <origin xyz="0.8891137 1.18206377 2.31900029"-->
+<!--                rpy="-0.10196342984026999 0.5145692159638564 -1.7990340284545345"/>-->
+<!--    </xacro:sensor_astra>-->
     <joint name="tool0-FT_sensor_base" type="fixed">
         <parent link="tool0"/>

Commit message: Fix robot xacro Co-authored-by: Pedro Amaral <pedromiglou.hotmail.com>

File: larcc_cell_description/urdf/larcc_cell.xacro (robot description, xacro)
@@ -38,22 +38,27 @@
 <!--    Place d45i camera-->
 <!--    Note: should add Pi value (3.14159) to second rotation value (p)-->
-    <xacro:realsense2_camera parent="world" use_nominal_extrinsics="true">
-<!--        <origin xyz="-0.161 0.222 1.210" rpy="3.210079633 2.720592654 2.809"/>-->
-        <origin xyz="-0.507 0.222 1.312" rpy="3.107 2.5559 -3.080"/>
-    </xacro:realsense2_camera>
-    <!-- Astra below was not well calibrated -->
-    <xacro:sensor_astra prefix="camera_4" parent="world">
+<!--    <xacro:realsense2_camera parent="world" use_nominal_extrinsics="true">-->
+<!--        <origin xyz="-0.507 0.222 1.312" rpy="3.107 2.5559 -3.080"/>-->
+<!--    </xacro:realsense2_camera>-->
+    <!-- Astra behind before calibration -->
+    <xacro:sensor_astra prefix="camera_behind" parent="world">
         <origin xyz="0.8891137 1.18206377 2.31900029"
-                rpy="-0.10196342984026999 0.5145692159638564 -1.7990340284545345"/>
+                rpy="-0.10196342984026999 2.08536416 -1.7990340284545345"/>
+        <!--                rpy="-0.10196342984026999 0.5145692159638564 -1.7990340284545345"/>-->
+    </xacro:sensor_astra>
+    <!-- Astra top before calibration -->
+    <xacro:sensor_astra prefix="camera_top" parent="world">
+        <origin xyz="0.1 0 2.41900029"
+                rpy="0 ${M_PI} 0"/>
     </xacro:sensor_astra>
     <joint name="tool0-FT_sensor_base" type="fixed">
         <parent link="tool0"/>
         <child link="FT_sensor_base"/>
-        <origin xyz="0 0 0.003" rpy="0 0 1.5708"/>
+        <origin xyz="0 0 0.007" rpy="0 0 ${M_PI/2}"/>
     </joint>
     <link name="FT_sensor_base">
         <visual>
           <geometry>
-            <cylinder length="0.006" radius="0.05"/>
+            <cylinder length="0.014" radius="0.05"/>
           </geometry>
           <material name="metalic_blue">
@@ -63,5 +68,5 @@
         <collision>
           <geometry>
-            <cylinder length="0.006" radius="0.05"/>
+            <cylinder length="0.014" radius="0.05"/>
           </geometry>
         </collision>
@@ -70,10 +75,10 @@
         <parent link="FT_sensor_base"/>
         <child link="FT_sensor"/>
-        <origin xyz="0 0 0.014" rpy="0 0 0"/>
+        <origin xyz="0 0 0.0215" rpy="0 0 0"/>
     </joint>
     <link name="FT_sensor">
         <visual>
           <geometry>
-            <cylinder length="0.022" radius="0.04"/>
+            <cylinder length="0.029" radius="0.04"/>
           </geometry>
           <material name="metalic_blue">
@@ -83,5 +88,5 @@
         <collision>
           <geometry>
-            <cylinder length="0.022" radius="0.04"/>
+            <cylinder length="0.029" radius="0.04"/>
           </geometry>
         </collision>
@@ -92,5 +97,5 @@
         <parent link="FT_sensor"/>
         <child link="robotiq_arg2f_base_link"/>
-        <origin xyz="0 0 0.011" rpy="0 0 0"/>
+        <origin xyz="0 0 0.0215" rpy="0 0 0"/>
     </joint>
     <link name="end_effector"/>
@@ -98,5 +103,5 @@
         <parent link="robotiq_arg2f_base_link"/>
         <child link="end_effector"/>
-        <origin xyz="0.0007295637845960989 0.0009607961805311316 0.21573113136562894" rpy="0 -0.001546440756787199 -1.572652377645297"/>
+        <origin xyz="0 0 0.21573113136562894" rpy="0 0 ${-M_PI/2}"/>
     </joint>
 <!--    Place base table-->

Commit message: temporary changes

File: larcc_cell_description/urdf/larcc_cell.xacro (robot description, xacro)
@@ -52,4 +52,9 @@
                 rpy="0 ${M_PI} 0"/>
     </xacro:sensor_astra>
+<!--    &lt;!&ndash; Astra top before calibration &ndash;&gt;-->
+<!--    <xacro:sensor_astra prefix="camera_gripper" parent="end_effector">-->
+<!--        <origin xyz="-0.12 -0.05 -0.1"-->
+<!--                rpy="${-M_PI/2} ${M_PI/8} 0"/>-->
+<!--    </xacro:sensor_astra>-->
     <joint name="tool0-FT_sensor_base" type="fixed">
         <parent link="tool0"/>

Commit message: cameras calibrated! Co-authored-by: Pedro-Amaral <pedromiglou@hotmail.com>

File: larcc_cell_description/urdf/larcc_cell.xacro (robot description, xacro)
@@ -39,16 +39,14 @@
 <!--    Note: should add Pi value (3.14159) to second rotation value (p)-->
 <!--    <xacro:realsense2_camera parent="world" use_nominal_extrinsics="true">-->
-<!--        <origin xyz="-0.507 0.222 1.312" rpy="3.107 2.5559 -3.080"/>-->
+<!--&lt;!&ndash;        <origin xyz="-0.507 0.222 1.312" rpy="3.107 2.5559 -3.080"/>&ndash;&gt;-->
+<!--        <origin xyz="-0.507 0.222 1.312" rpy="0.5640801120207652 0.03410154422820706 -1.8394088703112872"/>-->
 <!--    </xacro:realsense2_camera>-->
-    <!-- Astra behind before calibration -->
     <xacro:sensor_astra prefix="camera_behind" parent="world">
-        <origin xyz="0.8891137 1.18206377 2.31900029"
-                rpy="-0.10196342984026999 2.08536416 -1.7990340284545345"/>
-        <!--                rpy="-0.10196342984026999 0.5145692159638564 -1.7990340284545345"/>-->
+        <origin xyz="0.8481721310949765 1.224365708088931 2.3511875266550333"
+                rpy="-0.19718554582052114 0.5342533504487207 -1.8821968275695813"/>
     </xacro:sensor_astra>
-    <!-- Astra top before calibration -->
     <xacro:sensor_astra prefix="camera_top" parent="world">
-        <origin xyz="0.1 0 2.41900029"
-                rpy="0 0 0"/>
+        <origin xyz="0.09511408182797733 0.14905972847160784 2.4330682231422602"
+                rpy="-1.9962039976135075 1.491251777066553 -2.0400319820116386"/>
     </xacro:sensor_astra>
 <!--    &lt;!&ndash; Astra top before calibration &ndash;&gt;-->

Commit message: add a virtual ceiling to larccell_description

File: larcc_cell_description/urdf/larcc_cell.xacro (robot description, xacro)
@@ -122,3 +122,26 @@
         <origin xyz="${(0.9+0.7)/2} 0 0" rpy="0 0 0"/>
     </xacro:table_macro>
+     <!-- Collision box representing the ceiling -->
+    <link name="virtual_ceiling">
+      <collision>
+        <origin xyz="0 0 0.05" rpy="0 0 0"/>
+        <geometry>
+          <box size="5 5 0.1"/>
+        </geometry>
+      </collision>
+      <visual>
+        <origin xyz="0 0 0.05" rpy="0 0 0"/>
+        <geometry>
+          <box size="5 5 0.1"/>
+        </geometry>
+        <material name="red">
+          <color rgba="0.5 0 0 0.5"/>
+        </material>
+      </visual>
+    </link>
+    <joint name="fixed_ceiling_joint" type="fixed">
+      <parent link="world"/> <!-- Replace with your reference link -->
+      <child link="virtual_ceiling"/>
+      <origin xyz="0 0 1.8" rpy="0 0 0"/>
+    </joint>
 </robot>

Commit message: including wood block CAD model in larcc rviz and in robot model. including Socket communication client side (not yet fully working)

File: larcc_cell_description/urdf/larcc_cell.xacro (robot description, xacro)
@@ -25,4 +25,5 @@
     <xacro:include filename="$(find larcc_cell_description)/urdf/table.macro.xacro"/>
     <xacro:include filename="$(find larcc_cell_description)/urdf/gantry.macro.xacro"/>
+    <xacro:include filename="$(find larcc_cell_description)/urdf/wood_block.macro.xacro"/>
 <!--    Place gantry-->
     <xacro:gantry_macro name="gantry" parent="world" width="${gantry_width}"
@@ -52,9 +53,11 @@
                 rpy="-1.9962039976135075 1.491251777066553 -2.0400319820116386"/>
     </xacro:sensor_astra>
-<!--    &lt;!&ndash; Astra top before calibration &ndash;&gt;-->
-<!--    <xacro:sensor_astra prefix="camera_gripper" parent="end_effector">-->
-<!--        <origin xyz="-0.12 -0.05 -0.1"-->
-<!--                rpy="${-M_PI/2} ${M_PI/8} 0"/>-->
-<!--    </xacro:sensor_astra>-->
+    <xacro:sensor_astra prefix="camera_right" parent="world">
+        <origin xyz="-0.6 0.6 1.2"
+                rpy="0 0 0"/>
+    </xacro:sensor_astra>
+    <xacro:wood_block_macro parent="camera_right_rgb_optical_frame">
+        <origin xyz="-0.4 0.32 0.5" rpy="${M_PI/2} 0 0"/>
+    </xacro:wood_block_macro>
     <joint name="tool0-FT_sensor_base" type="fixed">
         <parent link="tool0"/>
@@ -136,5 +139,5 @@
         </geometry>
         <material name="red">
-          <color rgba="0.5 0 0 0.5"/>
+          <color rgba="0.5 0 0 0"/>
         </material>
       </visual>

Commit message: lar cell xacro update (with new table beam) cameras launch updated

File: larcc_cell_description/urdf/larcc_cell.xacro (robot description, xacro)
@@ -54,6 +54,6 @@
     </xacro:sensor_astra>
     <xacro:sensor_astra prefix="camera_right" parent="world">
-        <origin xyz="-0.6 0.6 1.2"
-                rpy="0 0 0"/>
+        <origin xyz="-0.45 0.6 1.46"
+                rpy="0 ${M_PI/6} ${-M_PI/4}"/>
     </xacro:sensor_astra>
     <xacro:wood_block_macro parent="camera_right_rgb_optical_frame">
@@ -125,4 +125,31 @@
         <origin xyz="${(0.9+0.7)/2} 0 0" rpy="0 0 0"/>
     </xacro:table_macro>
+    <link name="table_beam">
+        <visual>
+            <origin xyz="0.0 0.0 0.0" rpy="0 0 0" />
+            <geometry>
+                <mesh filename="package://larcc_cell_description/meshes/minitec_45x45_1500.STL" scale="0.001 0.001 0.001" />
+            </geometry>
+            <material name="grey"/>
+        </visual>
+        <collision>
+            <origin xyz="0 0 0" rpy="0 0 0" />
+            <geometry>
+                <box size="0.045 0.045 1.5"/>
+            </geometry>
+        </collision>
+        <inertial>
+            <mass value="1.0" />
+            <origin xyz="0.0 0.0 ${0.75/2-40-0.001}" rpy="0 0 0" />
+            <inertia ixx="0.1" ixy="0"  ixz="0"
+                     iyy="0.1" iyz="0"
+                     izz="0.01" />
+        </inertial>
+    </link>
+    <joint name="table_base_to_table_beam" type="fixed">
+        <parent link="table_base" />
+        <child link="table_beam" />
+        <origin xyz="0.305 -0.625 0.0025" rpy="${M_PI/2} 0 0"/>
+    </joint>
      <!-- Collision box representing the ceiling -->
     <link name="virtual_ceiling">

Commit message: lar cell xacro update, with new camera right intrinsic parameters (1280x780) and extrinsic parameters calibrated! Camera right is now fully working and ready to be used :)

File: larcc_cell_description/urdf/larcc_cell.xacro (robot description, xacro)
@@ -54,6 +54,6 @@
     </xacro:sensor_astra>
     <xacro:sensor_astra prefix="camera_right" parent="world">
-        <origin xyz="-0.45 0.6 1.46"
-                rpy="0 ${M_PI/6} ${-M_PI/4}"/>
+        <origin xyz="-0.48769570892652475 0.6173557198083176 1.2749729084453454"
+                rpy="0.23398734259638992 0.2798020805942116 -0.738576391893694"/>
     </xacro:sensor_astra>
     <xacro:wood_block_macro parent="camera_right_rgb_optical_frame">

Commit message: new right hand STL model added to larcc_cell.xacro. wood_block_client.py fully working now. Create wood_block_handover.launch for first big handover task trial

File: larcc_cell_description/urdf/larcc_cell.xacro (robot description, xacro)
@@ -26,4 +26,5 @@
     <xacro:include filename="$(find larcc_cell_description)/urdf/gantry.macro.xacro"/>
     <xacro:include filename="$(find larcc_cell_description)/urdf/wood_block.macro.xacro"/>
+    <xacro:include filename="$(find larcc_cell_description)/urdf/hand.macro.xacro"/>
 <!--    Place gantry-->
     <xacro:gantry_macro name="gantry" parent="world" width="${gantry_width}"
@@ -58,6 +59,9 @@
     </xacro:sensor_astra>
     <xacro:wood_block_macro parent="camera_right_rgb_optical_frame">
-        <origin xyz="-0.4 0.32 0.5" rpy="${M_PI/2} 0 0"/>
+        <origin xyz="0 0.25 0.7" rpy="${M_PI/2} 0 0"/>
     </xacro:wood_block_macro>
+    <xacro:hand_macro parent="camera_top_rgb_optical_frame">
+        <origin xyz="0 -0.1 1.5" rpy="0 ${-M_PI} 0"/>
+    </xacro:hand_macro>
     <joint name="tool0-FT_sensor_base" type="fixed">
         <parent link="tool0"/>

Commit message: removing right hand STL model adding minitec_45x45_1500.STL model (support of right camera) updating larcc_cell.xacro accordingly.

File: larcc_cell_description/urdf/larcc_cell.xacro (robot description, xacro)
@@ -26,5 +26,4 @@
     <xacro:include filename="$(find larcc_cell_description)/urdf/gantry.macro.xacro"/>
     <xacro:include filename="$(find larcc_cell_description)/urdf/wood_block.macro.xacro"/>
-    <xacro:include filename="$(find larcc_cell_description)/urdf/hand.macro.xacro"/>
 <!--    Place gantry-->
     <xacro:gantry_macro name="gantry" parent="world" width="${gantry_width}"
@@ -40,10 +39,4 @@
         <origin xyz="0 0 -0.015" rpy="0 0 0"/>
     </joint>
-<!--    Place d45i camera-->
-<!--    Note: should add Pi value (3.14159) to second rotation value (p)-->
-<!--    <xacro:realsense2_camera parent="world" use_nominal_extrinsics="true">-->
-<!--&lt;!&ndash;        <origin xyz="-0.507 0.222 1.312" rpy="3.107 2.5559 -3.080"/>&ndash;&gt;-->
-<!--        <origin xyz="-0.507 0.222 1.312" rpy="0.5640801120207652 0.03410154422820706 -1.8394088703112872"/>-->
-<!--    </xacro:realsense2_camera>-->
     <xacro:sensor_astra prefix="camera_behind" parent="world">
         <origin xyz="0.8481721310949765 1.224365708088931 2.3511875266550333"
@@ -61,7 +54,4 @@
         <origin xyz="0 0.25 0.7" rpy="${M_PI/2} 0 0"/>
     </xacro:wood_block_macro>
-    <xacro:hand_macro parent="camera_top_rgb_optical_frame">
-        <origin xyz="0 -0.1 1.5" rpy="0 ${-M_PI} 0"/>
-    </xacro:hand_macro>
     <joint name="tool0-FT_sensor_base" type="fixed">
         <parent link="tool0"/>

Commit message: First acceptable extrinsinc calibration between top camera and right camera. It is not perfect, but it suits, for now, the first handover task.

File: larcc_cell_description/urdf/larcc_cell.xacro (robot description, xacro)
@@ -39,8 +39,8 @@
         <origin xyz="0 0 -0.015" rpy="0 0 0"/>
     </joint>
-    <xacro:sensor_astra prefix="camera_behind" parent="world">
-        <origin xyz="0.8481721310949765 1.224365708088931 2.3511875266550333"
-                rpy="-0.19718554582052114 0.5342533504487207 -1.8821968275695813"/>
-    </xacro:sensor_astra>
+<!--    <xacro:sensor_astra prefix="camera_behind" parent="world">-->
+<!--        <origin xyz="0.8481721310949765 1.224365708088931 2.3511875266550333"-->
+<!--                rpy="-0.19718554582052114 0.5342533504487207 -1.8821968275695813"/>-->
+<!--    </xacro:sensor_astra>-->
     <xacro:sensor_astra prefix="camera_top" parent="world">
         <origin xyz="0.09511408182797733 0.14905972847160784 2.4330682231422602"
@@ -48,6 +48,6 @@
     </xacro:sensor_astra>
     <xacro:sensor_astra prefix="camera_right" parent="world">
-        <origin xyz="-0.48769570892652475 0.6173557198083176 1.2749729084453454"
-                rpy="0.23398734259638992 0.2798020805942116 -0.738576391893694"/>
+        <origin xyz="-0.47389933117248495 0.6050706033175103 1.2510900165155419"
+                rpy="0.1688160669718149 0.3885697035429511 -0.6796268633018927"/>
     </xacro:sensor_astra>
     <xacro:wood_block_macro parent="camera_right_rgb_optical_frame">

Commit message: velocity controller and larcc_cell.xacro updated

File: larcc_cell_description/urdf/larcc_cell.xacro (robot description, xacro)
@@ -51,6 +51,6 @@
                 rpy="0.1688160669718149 0.3885697035429511 -0.6796268633018927"/>
     </xacro:sensor_astra>
-    <xacro:wood_block_macro parent="camera_right_rgb_optical_frame">
-        <origin xyz="0 0.25 0.7" rpy="${M_PI/2} 0 0"/>
+    <xacro:wood_block_macro parent="world">
+        <origin xyz="0 0 0.86" rpy="0 0 ${M_PI}"/>
     </xacro:wood_block_macro>
     <joint name="tool0-FT_sensor_base" type="fixed">
